File: Spice/Testing.kicad_sch (KiCad schematic)
At the start: 9 parts, among them U1 74LS169

Commit message: update binary.cir
Parts:
- added R1: 10k, symbol Device:R
Connections:
- net GND: now also U1.8 (GND)
- net at U1.1 (U/~{D}): no longer V2.1
- net at U1.11 (Q3): now also R1.2
- net at U1.15 (~{TC}): now also R1.1
- net at U1.16 (VCC): now also V2.1
Other:
- note added: ".tran 0.1u 10m"
- note removed: ".tran 0.1u 200u"
- moved on the sheet: V2
Changed lines of the file:
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@@
 	(generator_version "9.0")
 	(paper "A4")
-	(text ".tran 0.1u 200u"
+	(text ".tran 0.1u 10m"
 		(exclude_from_sim no)
 		(at 142.24 43.434 0)
@@
 	)
 	(junction
+		(at 148.59 101.6)
+		(diameter 0)
+		(color 0 0 0 0)
+	)
+	(junction
 		(at 203.2 57.15)
 		(diameter 0)
@@
 	(wire
 		(pts
+			(xy 148.59 52.07) (xy 148.59 49.53)
+		)
+		(stroke
+			(width 0)
+			(type default)
+		)
+	)
+	(wire
+		(pts
 			(xy 191.77 67.31) (xy 203.2 67.31)
 		)
@@
 	(wire
 		(pts
-			(xy 116.84 69.85) (xy 114.3 69.85)
+			(xy 116.84 49.53) (xy 114.3 49.53)
 		)
 		(stroke
@@
 	(wire
 		(pts
-			(xy 128.27 69.85) (xy 128.27 77.47)
-		)
-		(stroke
-			(width 0)
-			(type default)
-		)
-	)
-	(wire
-		(pts
 			(xy 127 90.17) (xy 135.89 90.17)
 		)
@@
 	(wire
 		(pts
+			(xy 161.29 74.93) (xy 163.83 74.93)
+		)
+		(stroke
+			(width 0)
+			(type default)
+		)
+	)
+	(wire
+		(pts
 			(xy 114.3 90.17) (xy 114.3 101.6)
 		)
@@
 	(wire
 		(pts
+			(xy 148.59 101.6) (xy 181.61 101.6)
+		)
+		(stroke
+			(width 0)
+			(type default)
+		)
+	)
+	(wire
+		(pts
 			(xy 163.83 59.69) (xy 163.83 48.26)
 		)
@@
 	(wire
 		(pts
-			(xy 127 69.85) (xy 128.27 69.85)
-		)
-		(stroke
-			(width 0)
-			(type default)
-		)
-	)
-	(wire
-		(pts
-			(xy 114.3 69.85) (xy 114.3 90.17)
-		)
-		(stroke
-			(width 0)
-			(type default)
-		)
-	)
-	(wire
-		(pts
-			(xy 114.3 101.6) (xy 181.61 101.6)
-		)
-		(stroke
-			(width 0)
-			(type default)
-		)
-	)
-	(wire
-		(pts
-			(xy 128.27 77.47) (xy 135.89 77.47)
+			(xy 127 49.53) (xy 148.59 49.53)
+		)
+		(stroke
+			(width 0)
+			(type default)
+		)
+	)
+	(wire
+		(pts
+			(xy 114.3 49.53) (xy 114.3 90.17)
+		)
+		(stroke
+			(width 0)
+			(type default)
+		)
+	)
+	(wire
+		(pts
+			(xy 114.3 101.6) (xy 148.59 101.6)
 		)
 		(stroke
@@
 	(wire
 		(pts
+			(xy 163.83 67.31) (xy 161.29 67.31)
+		)
+		(stroke
+			(width 0)
+			(type default)
+		)
+	)
+	(wire
+		(pts
 			(xy 163.83 48.26) (xy 170.18 48.26)
 		)
@@
 		(pts
 			(xy 165.1 62.23) (xy 161.29 62.23)
+		)
+		(stroke
+			(width 0)
+			(type default)
+		)
+	)
+	(wire
+		(pts
+			(xy 148.59 97.79) (xy 148.59 101.6)
 		)
 		(stroke
@@
 			)
 		)
-		(property "Sim.Params" "y1=0 y2=5 td=0 tr=1u tf=1u tw=5u per=10u"
+		(property "Sim.Params" "y1=0 y2=5 td=10u tr=1u tf=1u tw=50u per=100u"
 			(at 122.0498 85.09 90)
 			(effects
@@
 			)
 		)
-		(property "Sim.Name" "counter3_ud"
+		(property "Sim.Name" "BIN4_COUNTER"
 			(at 148.59 74.93 0)
 			(effects
@@
 			)
 		)
-		(property "Sim.Pins" "1=ud 2=clk 12=b2 13=b1 14=b0"
+		(property "Sim.Pins" "2=CLK 11=Q3 12=Q2 13=Q1 14=Q0 15=RST"
 			(at 148.59 74.93 0)
 			(effects
@@
 	)
 	(symbol
+		(lib_id "Device:R")
+		(at 163.83 71.12 180)
+		(unit 1)
+		(exclude_from_sim no)
+		(in_bom yes)
+		(on_board yes)
+		(dnp no)
+		(fields_autoplaced yes)
+		(property "Reference" "R1"
+			(at 166.37 69.8499 0)
+			(effects
+				(font
+					(size 1.27 1.27)
+				)
+				(justify right)
+			)
+		)
+		(property "Value" "10k"
+			(at 166.37 72.3899 0)
+			(effects
+				(font
+					(size 1.27 1.27)
+				)
+				(justify right)
+			)
+		)
+		(property "Footprint" ""
+			(at 165.608 71.12 90)
+			(effects
+				(font
+					(size 1.27 1.27)
+				)
+				(hide yes)
+			)
+		)
+		(property "Datasheet" "~"
+			(at 163.83 71.12 0)
+			(effects
+				(font
+					(size 1.27 1.27)
+				)
+				(hide yes)
+			)
+		)
+		(property "Description" "Resistor"
+			(at 163.83 71.12 0)
+			(effects
+				(font
+					(size 1.27 1.27)
+				)
+				(hide yes)
+			)
+		)
+		(pin "1"
+		)
+		(pin "2"
+		)
+		(instances
+			(project "Testing"
+				(path "/3cc8ea43-d255-4f42-bfa7-b36af2da9d12"
+					(reference "R1")
+					(unit 1)
+				)
+			)
+		)
+	)
+	(symbol
 		(lib_id "Simulation_SPICE:VDC")
-		(at 121.92 69.85 270)
+		(at 121.92 49.53 270)
 		(unit 1)
 		(exclude_from_sim no)
@@
 		(fields_autoplaced yes)
 		(property "Reference" "V2"
-			(at 122.0498 62.23 90)
+			(at 122.0498 41.91 90)
 			(effects
 				(font
@@
 		)
 		(property "Value" "5"
-			(at 122.0498 64.77 90)
+			(at 122.0498 44.45 90)
 			(effects
 				(font
@@
 		)
 		(property "Footprint" ""
-			(at 121.92 69.85 0)
+			(at 121.92 49.53 0)
 			(effects
 				(font
@@
 		)
 		(property "Datasheet" "https://ngspice.sourceforge.io/docs/ngspice-html-manual/manual.xhtml#sec_Independent_Sources_for"
-			(at 121.92 69.85 0)
+			(at 121.92 49.53 0)
 			(effects
 				(font
@@
 		)
 		(property "Description" "Voltage source, DC"
-			(at 121.92 69.85 0)
+			(at 121.92 49.53 0)
 			(effects
 				(font
@@
 		)
 		(property "Sim.Pins" "1=+ 2=-"
-			(at 121.92 69.85 0)
+			(at 121.92 49.53 0)
 			(effects
 				(font
@@
 		)
 		(property "Sim.Type" "DC"
-			(at 121.92 69.85 0)
+			(at 121.92 49.53 0)
 			(effects
 				(font
@@
 		)
 		(property "Sim.Device" "V"
-			(at 121.92 69.85 0)
-			(effects
-				(font
+			(at 121.92 49.53 0)
+			(effects
+				(font
