File: Spice/_autosave-Testing.kicad_sch (KiCad schematic)
At the start: 12 parts, among them U1 SN74HC161DR

Commit message: Binary Update
Parts:
- added U2: 74LS393, symbol 74xx:74LS393
Changed lines of the file:
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@@
+	)
+	(symbol
+		(lib_id "74xx:74LS393")
+		(at 76.2 74.93 0)
+		(unit 1)
+		(exclude_from_sim no)
+		(in_bom yes)
+		(on_board yes)
+		(dnp no)
+		(fields_autoplaced yes)
+		(property "Reference" "U2"
+			(at 76.2 64.77 0)
+			(effects
+				(font
+					(size 1.27 1.27)
+				)
+			)
+		)
+		(property "Value" "74LS393"
+			(at 76.2 67.31 0)
+			(effects
+				(font
+					(size 1.27 1.27)
+				)
+			)
+		)
+		(property "Footprint" ""
+			(at 76.2 74.93 0)
+			(effects
+				(font
+					(size 1.27 1.27)
+				)
+				(hide yes)
+			)
+		)
+		(property "Datasheet" "74xx\\74LS393.pdf"
+			(at 76.2 74.93 0)
+			(effects
+				(font
+					(size 1.27 1.27)
+				)
+				(hide yes)
+			)
+		)
+		(property "Description" "Dual BCD 4-bit counter"
+			(at 76.2 74.93 0)
+			(effects
+				(font
+					(size 1.27 1.27)
+				)
+				(hide yes)
+			)
+		)
+		(pin "10"
+		)
+		(pin "14"
+		)
+		(pin "3"
+		)
+		(pin "4"
+		)
+		(pin "9"
+		)
+		(pin "2"
+		)
+		(pin "12"
+		)
+		(pin "13"
+		)
+		(pin "5"
+		)
+		(pin "1"
+		)
+		(pin "11"
+		)
+		(pin "6"
+		)
+		(pin "8"
+		)
+		(pin "7"
+		)
+		(instances
+			(project ""
+				(path "/3cc8ea43-d255-4f42-bfa7-b36af2da9d12"
+					(reference "U2")
+					(unit 1)
+				)
+			)
+		)
 	)
 	(symbol
@@
 			)
 		)
-		(property "Sim.Params" "vcc1=5 speed1=1 tripdt1=0"
-			(at 124.46 54.61 0)
-			(effects
+		(property "Sim.Params" "vcc1=5V speed1=1 tripdt1=0"
+			(at 124.46 54.61 0)
+			(effects
