File: Spice/capSensorReader.kicad_sch (KiCad schematic)
At the start: 15 parts, among them U1 LM358, U2 LM358

Commit message: Redo Base Project file add code
Changed lines of the file:
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@@
 			)
 		)
-		(property "Sim.Params" "dc=0 ampl=.1 f=100k ac=0"
+		(property "Sim.Params" "dc=0 ampl=.1 f=300k ac=0"
 			(at 92.71 119.126 0)
 			(effects
