File: Spice/capSensorReader.kicad_sch (KiCad schematic)
At the start: 30 parts, among them U1 LM358, U2 LM358, U3 LM358

Commit message: Better Sensor Reader
Parts:
- removed C6: 787nF, symbol Device:C
- removed D2, D3, D4: 1N34A, Diode_THT:D_DO-35_SOD27_P2.54mm_Vertical_AnodeUp, symbol Device:D
- removed R2, R3: 1k, symbol Device:R
- removed R4: 6.19k, symbol Device:R
- removed R5: 4.22k, symbol Device:R
- removed R6: 6.98k, symbol Device:R
- removed U3: LM358, symbol Amplifier_Operational:LM358
- added Rc2, Rc4: 100k, symbol Device:R
- added Rc3, Rc5: 1k, symbol Device:R
- C1: value 8p -> 3p
- C3, C4: value 75p -> 100p
- C5: value 100nF -> 100p
- Cf1: value 2p -> 10p
Connections:
- net GND: now also C5.2
- net at C5.1: now also D1.1 (K), Rc2.1
- net at U1.5 (+): now also Rc4.2, Rc5.2; no longer C5.2
- net at C3.1: now also Rc3.1
- net at Rc1.2, U1.1: no longer D1.2 (A)
- net at C4.1: now also Rc5.1
- new net: Rc2.2, Rc3.2, Rc4.1
Other:
- moved on the sheet: R1, Rd1, U1B, U2A, U2B, Vin1
