File: Spice/_autosave-capSensorReader.kicad_sch (KiCad schematic)
At the start: 30 parts, among them U1 LM358, U2 LM358, U3 LM358

Commit message: Added rectifier and passive low-pass filter (RC)
Parts:
- removed C5: 100nF, symbol Device:C
- removed C6: 787nF, symbol Device:C
- removed D2, D3, D4: 1N34A, Diode_THT:D_DO-35_SOD27_P2.54mm_Vertical_AnodeUp, symbol Device:D
- removed R5: 4.22k, symbol Device:R
- removed R6: 6.98k, symbol Device:R
- removed U3: LM358, symbol Amplifier_Operational:LM358
- R4: value 6.19k -> 6k
Connections:
- net at U1.5 (+): now also C4.1, R3.2
- net at R2.1: now also R4.2
- no-connect marks 3 -> 0
Other:
- moved on the sheet: C3, C4, R1, R2, R3, U1B
