File: Hierarchical Sheets/8xAmplifier.kicad_sch (KiCad schematic)
At the start: 0 parts

Commit message: remove Hierarchical Sheets folder inside Hierarchical Sheets foler
Other:
- sheet Amplifier: file ./Hierarchical Sheets/amplifier.kicad_sch -> amplifier.kicad_sch
- sheet Amplifier1: file Hierarchical Sheets/amplifier.kicad_sch -> amplifier.kicad_sch
- sheet Amplifier2: file Hierarchical Sheets/amplifier.kicad_sch -> amplifier.kicad_sch
- sheet Amplifier3: file Hierarchical Sheets/amplifier.kicad_sch -> amplifier.kicad_sch
- sheet Amplifier4: file Hierarchical Sheets/amplifier.kicad_sch -> amplifier.kicad_sch
- sheet Amplifier5: file Hierarchical Sheets/amplifier.kicad_sch -> amplifier.kicad_sch
- sheet Amplifier6: file Hierarchical Sheets/amplifier.kicad_sch -> amplifier.kicad_sch
- sheet Amplifier7: file Hierarchical Sheets/amplifier.kicad_sch -> amplifier.kicad_sch
Changed lines of the file:
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@@
 			)
 		)
-		(property "Sheetfile" "Hierarchical Sheets/amplifier.kicad_sch"
+		(property "Sheetfile" "amplifier.kicad_sch"
 			(at 146.05 38.6846 0)
 			(effects
@@
 			)
 		)
-		(property "Sheetfile" "Hierarchical Sheets/amplifier.kicad_sch"
+		(property "Sheetfile" "amplifier.kicad_sch"
 			(at 146.05 89.4846 0)
 			(effects
@@
 			)
 		)
-		(property "Sheetfile" "Hierarchical Sheets/amplifier.kicad_sch"
+		(property "Sheetfile" "amplifier.kicad_sch"
 			(at 146.05 64.0846 0)
 			(effects
@@
 			)
 		)
-		(property "Sheetfile" "Hierarchical Sheets/amplifier.kicad_sch"
+		(property "Sheetfile" "amplifier.kicad_sch"
 			(at 101.6 114.8846 0)
 			(effects
@@
 			)
 		)
-		(property "Sheetfile" "Hierarchical Sheets/amplifier.kicad_sch"
+		(property "Sheetfile" "amplifier.kicad_sch"
 			(at 101.6 38.6846 0)
 			(effects
@@
 			)
 		)
-		(property "Sheetfile" "Hierarchical Sheets/amplifier.kicad_sch"
+		(property "Sheetfile" "amplifier.kicad_sch"
 			(at 101.6 89.4846 0)
 			(effects
@@
 			)
 		)
-		(property "Sheetfile" "./Hierarchical Sheets/amplifier.kicad_sch"
+		(property "Sheetfile" "amplifier.kicad_sch"
 			(at 101.6 64.0846 0)
 			(effects
@@
 			)
 		)
-		(property "Sheetfile" "Hierarchical Sheets/amplifier.kicad_sch"
+		(property "Sheetfile" "amplifier.kicad_sch"
 			(at 146.05 114.8846 0)
 			(effects
