File: capstone_oscillator.kicad_sch (KiCad schematic)
At the start: 6 parts, among them U1 LMC555xM, U2 CD4018BE

Commit message: continued work on osc/logic circuit
Parts:
- added U3: CD4011BM96, D14, symbol CD4011BM96:CD4011BM96
Connections:
- net GND: now also U2.12 (JAM5), U2.15 (RESET), U2.2 (JAM1), U2.3 (JAM2), U2.7 (JAM3), U2.9 (JAM4)
- net at U2.1 (DATA): now also U3.9 (J)
- net at U2.4 (*Q2): now also U3.1 (A)
- net at U2.6 (*Q3): now also U3.2 (B)
Other:
- moved on the sheet: U2

Commit message: timer oscillator
Parts:
- added U4: CD74HCT175E, N16, symbol CD74HCT175E:CD74HCT175E
- added V1: 5, symbol Simulation_SPICE:VDC
- C1: value C -> .1u
- C3: value C -> 300n
- R1: value R -> 1k
- Rc1: renamed from Rc; value R -> 10k
Connections:
- net GND: now also U1.5 (CONT), U2.10 (PRESETENABLE), U2.8 (VSS), U4.8 (GND), V1.2
- net OUTPUT: now also U4.3 (*Q0); no longer C1.1, R1.1, Rc1.1, U1.3 (OUT), U1.4 (~{RST}), U1.8 (VCC)
- net at U2.1 (DATA): now also U2.13 (*Q5); no longer U3.9 (J)
- net +5VDC: now reaches U2.16 (VDD)
- new net: U4.2 (Q0), U4.4 (D0)
- new net Vs: C1.1, R1.1, Rc1.1, U1.3 (OUT), U1.4 (~{RST}), U1.8 (VCC), V1.1
Other:
- note added: "Crystal Oscillator IC - 50% duty cycle @ 3MHz"
- note added: "Divide-by-N counter - configured as divide-by-5 - 3Mhz -> 600kHz"
- note added: "NAND gate for divide-by-5 configuration"
- note added: "flip-flop - divide-by-2 - output : 50% duty cycle @ 300kHz"
- moved on the sheet: C1, C3, R1, Rc1, U1, U2, U3
